Commit message: Added basic simulation code

File: bb_description/urdf/jessi.urdf (robot description, URDF)
Before this commit: robot Jessii, 12 links, 11 joints
Links:
- removed link axle
- removed link base_footprint
- removed link front_ball
- removed link gps
- removed link imu
- removed link left_wheel
- removed link lidar
- removed link magnetometer
- removed link optical_cam_center
- removed link right_wheel
- removed link usb_cam_center
- added link ackermann_bar_link, mass 0.01; collision box size=0.015 0.15 0.01; visual box size=0.015 0.15 0.01
- added link back_left_wheel_link, mass 0.01; collision cylinder length=0.025 radius=0.06; visual cylinder length=0.025 radius=0.06
- added link back_right_wheel_link, mass 0.01; collision cylinder length=0.025 radius=0.06; visual cylinder length=0.025 radius=0.06
- added link base_scan_link, mass 0.1; collision cylinder length=0.028 radius=0.0229; visual cylinder length=0.028 radius=0.0229
- added link front_left_bar_link, mass 0.01; collision box size=0.03 0.01995 0.005; visual box size=0.03 0.01995 0.005
- added link front_left_wheel_link, mass 0.01; collision cylinder length=0.025 radius=0.06; visual cylinder length=0.025 radius=0.06
- added link front_link, mass 0.01; collision box size=0.015 0.15 0.005; visual box size=0.015 0.15 0.005
- added link front_right_bar_link, mass 0.01; collision box size=0.03 0.01995 0.005; visual box size=0.03 0.01995 0.005
- added link front_right_wheel_link, mass 0.01; collision cylinder length=0.025 radius=0.06; visual cylinder length=0.025 radius=0.06
- added link laser_base_link, mass 0.1; collision box size=0.05 0.05 0.05; visual box size=0.05 0.05 0.05
- added link steer_link, mass 0.01; collision box size=0.03 0.01995 0.005; visual box size=0.03 0.01995 0.005
- link base_link: mass None -> 0.2; geometry collision box size=0.3 0.15 0.1; visual box size=0.3 0.15 0.1
Joints:
- removed joint axle_to_left_wheel
- removed joint axle_to_right_wheel
- removed joint base_footprint_to_axle
- removed joint base_footprint_to_base_link
- removed joint base_footprint_to_center_camera
- removed joint base_footprint_to_front_ball
- removed joint base_footprint_to_gps
- removed joint base_footprint_to_imu
- removed joint base_footprint_to_lidar
- removed joint base_footprint_to_magnetometer
- removed joint optical_cam_center_joint
- added joint ackermann_joint: type revolute, parent steer_link, child ackermann_bar_link, origin xyz=-0.04 0 0 rpy=0 0 0, axis 0 0 1, limit lower=-0.5 upper=0.5 effort=100 velocity=10
- added joint back_left_wheel_joint: type continuous, parent base_link, child back_left_wheel_link, origin xyz=-0.16 0.1 -0.1 rpy=0 0 0, axis 0 1 0
- added joint back_right_wheel_joint: type continuous, parent base_link, child back_right_wheel_link, origin xyz=-0.16 -0.1 -0.1 rpy=0 0 0, axis 0 1 0
- added joint base_scan_joint: type fixed, parent laser_base_link, child base_scan_link, origin xyz=0 0 0.05 rpy=0 0 0
- added joint front_joint: type fixed, parent base_link, child front_link, origin xyz=0.16 0.0 -0.1
- added joint front_left_bar_joint: type revolute, parent front_link, child front_left_bar_link, origin xyz=0.0 0.06 0.0 rpy=0 0 0, axis 0 0 1, limit lower=-0.5 upper=0.5 effort=100 velocity=10
- added joint front_left_wheel_joint: type continuous, parent front_left_bar_link, child front_left_wheel_link, origin xyz=0 0.04 0 rpy=0 0 0, axis 0 1 0
- added joint front_right_bar_joint: type revolute, parent front_link, child front_right_bar_link, origin xyz=0.0 -0.06 0.0 rpy=0 0 0, axis 0 0 1, limit lower=-0.5 upper=0.5 effort=100 velocity=10
- added joint front_right_wheel_joint: type continuous, parent front_right_bar_link, child front_right_wheel_link, origin xyz=0 -0.04 0 rpy=0 0 0, axis 0 1 0
- added joint laser_base_mount_joint: type fixed, parent base_link, child laser_base_link, origin xyz=0 0 0.05 rpy=0 0 0
- added joint steer_joint: type revolute, parent front_link, child steer_link, origin xyz=0.0 0.0 0.0 rpy=0 0 0, axis 0 0 1, limit lower=-0.5 upper=0.5 effort=100 velocity=10

File: bb_description/urdf/jessii.urdf.xacro (robot description, xacro)
@@ -7,5 +7,5 @@
   <!-- constants -->
   <xacro:property name="M_PI" value="3.1415926535897931" />
-  <xacro:property name="chassis_mass" value="20" />
+  <xacro:property name="chassis_mass" value="32" />
   <!-- wheels -->
   <xacro:property name="drive_tire_diameter" value="0.305"/>
@@ -22,44 +22,4 @@
   <xacro:property name="drive_shock_eff_limit" value="500.0"/>
   <xacro:property name="drive_shock_vel_limit" value="0.1"/>
-  <!-- casters -->
-  <xacro:property name="caster_radius" value="0.1016"/>
-  <xacro:property name="caster_mass" value="1.0"/>
-  <!-- how far forward from base_link it is -->
-  <xacro:property name="caster_x" value="0.612978"/>
-  <!-- center camera params, relative to the magnetometer -->
-  <xacro:property name="center_camera_y" value="0.0"/>
-  <xacro:property name="center_camera_x" value="0.0"/>
-  <xacro:property name="center_camera_pitch" value="0.418879"/>
-  <xacro:property name="center_camera_z" value="0.043942"/>
-  <!-- right camera params, relative to the magnetometer -->
-  <xacro:property name="right_camera_y" value="-0.33147"/>
-  <xacro:property name="right_camera_x" value="0.019812"/>
-  <xacro:property name="right_camera_pitch" value="1.06465"/>
-  <xacro:property name="right_camera_yaw" value="-1.13446"/>
-  <xacro:property name="right_camera_z" value="0"/>
-  <!-- left camera params, relative to the magnetometer -->
-  <xacro:property name="left_camera_y" value="0.33147"/>
-  <xacro:property name="left_camera_x" value="0.019812"/>
-  <xacro:property name="left_camera_pitch" value="1.06465"/>
-  <xacro:property name="left_camera_yaw" value="1.13446"/>
-  <xacro:property name="left_camera_z" value="0.0"/>
-  <!-- lidar params relative to base_link-->
-  <xacro:property name="lidar_pitch" value="0.174533"/>
-  <xacro:property name="lidar_x" value="0.680364"/>
-  <xacro:property name="lidar_z" value="0.237121"/>
-  <xacro:property name="lidar_hz" value="10"/>
-  <xacro:property name="lidar_samples" value="500"/>
-  <!-- gps, relative to base_link -->
-  <xacro:property name="gps_z" value="1.354330"/>
-  <xacro:property name="gps_y" value="0.198120"/>
-  <xacro:property name="gps_x" value="0.216371"/>
-  <!-- imu bottom, relative to base_link -->
-  <xacro:property name="imu_z" value="0.221742"/>
-  <xacro:property name="imu_y" value="0.0"/>
-  <xacro:property name="imu_x" value="-0.024638"/>
-  <!-- imu top, relative to base_link -->
-  <xacro:property name="magnetometer_z" value="1.238758"/>
-  <xacro:property name="magnetometer_y" value="0.0"/>
-  <xacro:property name="magnetometer_x" value="0.216371"/>
   <!-- gives small geometry so it show up in rviz -->
   <xacro:macro name="null_link">
@@ -74,507 +34,48 @@
     </visual>
   </xacro:macro>
-  <!-- makes shock for drive wheel -->
-  <xacro:macro name="drive_shock"
-               params="lr_prefix lr_reflect">
-    <joint name="${lr_prefix}_drive_shock" type="prismatic">
-      <parent link="base_link"/>
-      <child link="${lr_prefix}_axle_carrier"/>
-      <origin xyz="0 ${lr_reflect * wheelbase / 2} 0"
-              rpy="0 0 0"/>
-      <axis xyz="0 0 -1"/>
-      <limit lower="${-drive_wheel_travel / 2}" upper="${drive_wheel_travel / 2}"
-             effort="${drive_shock_eff_limit}" velocity="${drive_shock_vel_limit}"/>
-      <!-- TODO tune for actual shocks -->
-      <!-- damping = viscous dampening coeff -->
-      <!-- friction, physical static friction -->
-      <!-- spring stiffness = spring constant N/m-->
-      <dynamics damping="100" friction="1.0"
-                spring_stiffness="113832.44275" spring_reference="0.08"/>
-    </joint>
-    <transmission name="${lr_prefix}_drive_shock_trans">
-      <type>transmission_interface/SimpleTransmission</type>
-      <joint name="${lr_prefix}_drive_shock">
-        <hardwareInterface>hardware_interface/EffortJointInterface</hardwareInterface>
-      </joint>
-      <actuator name="${lr_prefix}_drive_shock_act">
-        <!-- This hardwareInterface element exists for compatibility
-             with ROS Hydro. -->
-        <hardwareInterface>hardware_interface/EffortJointInterface</hardwareInterface>
-        <!-- TODO parameterize to make consistent PID values work -->
-        <mechanicalReduction>1</mechanicalReduction>
-      </actuator>
-    </transmission>
-  </xacro:macro>
-  <!-- The "wheel" macro defines an axle carrier, axle, and wheel. -->
-  <xacro:macro name="wheel" params="lr_prefix lr_reflect tire_diameter wheel_mass axle_eff_limit wheel_width">
-    <link name="${lr_prefix}_axle_carrier">
-      <xacro:null_link/>
-    </link>
-    <!-- The left and right axles have the same axis so that identical
-         rotation values cause the wheels to rotate in the same direction. -->
-    <joint name="${lr_prefix}_axle" type="continuous">
-      <parent link="${lr_prefix}_axle_carrier"/>
-      <child link="${lr_prefix}_wheel"/>
-      <origin xyz="0 0 0" rpy="${M_PI / 2} 0 0"/>
-      <axis xyz="0 0 -1"/>
-      <limit effort="${drive_wheel_eff_limit}" velocity="${drive_wheel_vel_limit}"/>
-      <dynamics damping="0.001" friction="0.5"/>
-    </joint>
-    <transmission name="${lr_prefix}_axle_trans">
-      <type>transmission_interface/SimpleTransmission</type>
-      <joint name="${lr_prefix}_axle">
-        <hardwareInterface>hardware_interface/EffortJointInterface</hardwareInterface>
-      </joint>
-      <actuator name="${lr_prefix}_axle_act">
-        <!--This hardwareInterface element exists for compatibility
-             with ROS Hydro-->
-        <hardwareInterface>hardware_interface/EffortJointInterface</hardwareInterface>
-        <mechanicalReduction>1</mechanicalReduction>
-      </actuator>
-    </transmission>
-    <link name="${lr_prefix}_wheel">
-      <visual>
-        <geometry>
-          <mesh filename="package://igvc_description/urdf/meshes/Wheel.dae"/>
-        </geometry>
-      </visual>
-      <collision>
-        <geometry>
-          <mesh filename="package://igvc_description/urdf/meshes/Wheel.dae"/>
-        </geometry>
-        <max_contacts>10</max_contacts>
-        <surface>
-          <contact>
-            <ode>
-              <soft_cfm>0.000000001</soft_cfm>
-              <soft_erp>0.2</soft_erp>
-              <kp>1e+10</kp>
-              <kd>10</kd>
-              <max_vel>0.01</max_vel>
-              <min_depth>0.005</min_depth>
-            </ode>
-          </contact>
-        </surface>
-      </collision>
-      <inertial>
-        <origin xyz="0 0 0" />
-        <mass value="${wheel_mass}"/>
-        <inertia  ixx="${1 / 12 * wheel_mass * wheel_width**2 + 1/4 * wheel_mass * (tire_diameter / 2)**2}"
-                  ixy="0.0"
-                  ixz="0.0"
-                  iyy="${1 / 12 * wheel_mass * wheel_width**2 + 1/4 * wheel_mass * (tire_diameter / 2)**2}"
-                  iyz="0.0"
-                  izz="${1/2 * wheel_mass * (tire_diameter / 2)**2}" />
-      </inertial>
-    </link>
-    <xacro:drive_shock lr_prefix="${lr_prefix}" lr_reflect="${lr_reflect}"/>
-    <gazebo reference="${lr_prefix}_wheel">
-      <mu1>0.7</mu1>
-      <mu2>0.75</mu2>
-    </gazebo>
-  </xacro:macro>
-  <!-- macro used to define casters -->
-  <xacro:macro name="caster" params="ball_radius ball_mass tire_diameter x y">
-    <link name="caster">
-      <inertial>
-        <mass value="${ball_mass}" />
-        <origin xyz="0 0 0" rpy="0 0 0"/>
-        <inertia  ixx="${2 / 5 * ball_mass * ball_radius ** 2}" ixy="0.0" ixz="0.0"
-                  iyy="${2 / 5 * ball_mass * ball_radius ** 2}" iyz="0.0"
-                  izz="${2 / 5 * ball_mass * ball_radius ** 2}" />
-      </inertial>
-      <visual>
-        <geometry>
-          <sphere radius="${ball_radius}"/>
-        </geometry>
-      </visual>
-      <collision>
-        <geometry>
-          <sphere radius="${ball_radius}"/>
-        </geometry>
-      </collision>
-    </link>
-    <joint name="base_link_to_caster" type="fixed">
-      <parent link="base_link"/>
-      <child link="caster"/>
-      <origin xyz="${x} ${y} ${ball_radius - tire_diameter / 2}" rpy="0 0 0"/>
-    </joint>
-    <gazebo reference="caster">
-      <mu1>0.2</mu1>
-      <mu2>0.25</mu2>
-    </gazebo>
-    <gazebo>
-      <joint name='base_link_to_caster' type='ball'>
-        <parent>base_link</parent>
-        <child>caster</child>
-        <pose frame=''>0 0 0 0 0 0</pose>
-        <physics>
-          <ode>
-            <limit>
-              <cfm>0</cfm>
-              <erp>0.2</erp>
-            </limit>
-            <suspension>
-              <cfm>0</cfm>
-              <erp>0.2</erp>
-            </suspension>
-          </ode>
-        </physics>
-      </joint>
-    </gazebo>
-  </xacro:macro>
-  <link name="cam/center">
-      <visual>
-          <geometry>
-              <box size="0.1 0.1 0.1"/>
-          </geometry>
-      </visual>
-  </link>
-  <joint name="magnetometer_to_center_cam" type="fixed">
-      <origin xyz="${center_camera_x} ${center_camera_y} ${center_camera_z}" rpy="0 ${center_camera_pitch} 0" />
-      <parent link="magnetometer"/>
-      <child link="cam/center"/>
-  </joint>
-  <!-- the optical joint is in the correct frame for transforms -->
-  <link name="cam/center_optical"/>
-  <joint name="cam/center_optical_joint" type="fixed">
-      <parent link="cam/center"/>
-      <child link="cam/center_optical"/>
-      <origin xyz="0 0 0" rpy="-1.5708 0 -1.5708"/>
-  </joint>
-  <gazebo reference="cam/center">
-      <sensor name="center_cam_sensor" type="camera">
-          <camera>
-              <!-- hov in radians -->
-              <horizontal_fov>1.2290609</horizontal_fov>
-              <image>
-                <width>1920</width>
-                <height>1080</height>
-              </image>
-              <clip>
-                <near>0.1</near>
-                <far>100</far>
-              </clip>
-              <!--
-                  <distortion>
-                  <k1>-0.25</k1>
-                  <k2>0.12</k2>
-                  <k3>0.0</k3>
-                  <p1>-0.00028</p1>
-                  <p2>-0.00005</p2>
-                  <center>0.5 0.5</center>
-                  </distortion>
-              -->
-          </camera>
-          <always_on>1</always_on>
-          <update_rate>30</update_rate>
-          <plugin name="camera_controller" filename="libgazebo_ros_camera.so">
-              <alwaysOn>true</alwaysOn>
-              <updateRate>30</updateRate>
-              <cameraName>cam/center/raw</cameraName>
-              <imageTopicName>image</imageTopicName>
-              <cameraInfoTopicName>camera_info</cameraInfoTopicName>
-              <frameName>cam/center_optical</frameName>
-              <hackBaseline>0.0</hackBaseline>
-              <distortionK1>0.0</distortionK1>
-              <distortionK2>0.0</distortionK2>
-              <distortionK3>0.0</distortionK3>
-              <distortionT1>0.0</distortionT1>
-              <distortionT2>0.0</distortionT2>
-          </plugin>
-      </sensor>
-  </gazebo>
-  <link name="cam/right">
-      <visual>
-          <geometry>
-              <box size="0.1 0.1 0.1"/>
-          </geometry>
-      </visual>
-  </link>
-  <joint name="magnetometer_to_right_cam" type="fixed">
-      <origin xyz="${right_camera_x} ${right_camera_y} ${right_camera_z}" rpy="0 ${right_camera_pitch} ${right_camera_yaw}" />
-      <parent link="magnetometer"/>
-      <child link="cam/right"/>
-  </joint>
-  <!-- the optical joint is in the correct frame for transforms -->
-  <link name="cam/right_optical"/>
-  <joint name="cam/right_optical_joint" type="fixed">
-      <parent link="cam/right"/>
-      <child link="cam/right_optical"/>
-      <origin xyz="0 0 0" rpy="-1.5708 0 -1.5708"/>
-  </joint>
-  <gazebo reference="cam/right">
-      <sensor name="right_cam_sensor" type="camera">
-          <camera>
-              <!-- hov in radians -->
-              <horizontal_fov>1.2290609</horizontal_fov>
-              <image>
-                <width>1920</width>
-                <height>1080</height>
-              </image>
-              <clip>
-                <near>0.1</near>
-                <far>100</far>
-              </clip>
-              <!--
-                  <distortion>
-                  <k1>-0.25</k1>
-                  <k2>0.12</k2>
-                  <k3>0.0</k3>
-                  <p1>-0.00028</p1>
-                  <p2>-0.00005</p2>
-                  <center>0.5 0.5</center>
-                  </distortion>
-              -->
-          </camera>
-          <always_on>1</always_on>
-          <update_rate>30</update_rate>
-          <plugin name="camera_controller" filename="libgazebo_ros_camera.so">
-              <alwaysOn>true</alwaysOn>
-              <updateRate>30</updateRate>
-              <cameraName>cam/right/raw</cameraName>
-              <imageTopicName>image</imageTopicName>
-              <cameraInfoTopicName>camera_info</cameraInfoTopicName>
-              <frameName>cam/right_optical</frameName>
-              <hackBaseline>0.0</hackBaseline>
-              <distortionK1>0.0</distortionK1>
-              <distortionK2>0.0</distortionK2>
-              <distortionK3>0.0</distortionK3>
-              <distortionT1>0.0</distortionT1>
-              <distortionT2>0.0</distortionT2>
-          </plugin>
-      </sensor>
-  </gazebo>
-  <link name="cam/left">
-      <visual>
-          <geometry>
-              <box size="0.1 0.1 0.1"/>
-          </geometry>
-      </visual>
-  </link>
-  <joint name="magnetometer_to_left_cam" type="fixed">
-      <origin xyz="${left_camera_x} ${left_camera_y} ${left_camera_z}" rpy="0 ${left_camera_pitch} ${left_camera_yaw}" />
-      <parent link="magnetometer"/>
-      <child link="cam/left"/>
-  </joint>
-  <!-- the optical joint is in the correct frame for transforms -->
-  <link name="cam/left_optical"/>
-  <joint name="cam/left_optical_joint" type="fixed">
-      <parent link="cam/left"/>
-      <child link="cam/left_optical"/>
-      <origin xyz="0 0 0" rpy="-1.5708 0 -1.5708"/>
-  </joint>
-  <gazebo reference="cam/left">
-      <sensor name="left_cam_sensor" type="camera">
-          <camera>
-              <!-- hov in radians -->
-              <horizontal_fov>1.2290609</horizontal_fov>
-              <image>
-                <width>1920</width>
-                <height>1080</height>
-              </image>
-              <clip>
-                <near>0.1</near>
-                <far>100</far>
-              </clip>
-              <!--
-                  <distortion>
-                  <k1>-0.25</k1>
-                  <k2>0.12</k2>
-                  <k3>0.0</k3>
-                  <p1>-0.00028</p1>
-                  <p2>-0.00005</p2>
-                  <center>0.5 0.5</center>
-                  </distortion>
-              -->
-          </camera>
-          <always_on>1</always_on>
-          <update_rate>30</update_rate>
-          <plugin name="camera_controller" filename="libgazebo_ros_camera.so">
-              <alwaysOn>true</alwaysOn>
-              <updateRate>30</updateRate>
-              <cameraName>cam/left/raw</cameraName>
-              <imageTopicName>image</imageTopicName>
-              <cameraInfoTopicName>camera_info</cameraInfoTopicName>
-              <frameName>cam/left_optical</frameName>
-              <hackBaseline>0.0</hackBaseline>
-              <distortionK1>0.0</distortionK1>
-              <distortionK2>0.0</distortionK2>
-              <distortionK3>0.0</distortionK3>
-              <distortionT1>0.0</distortionT1>
-              <distortionT2>0.0</distortionT2>
-          </plugin>
-      </sensor>
-  </gazebo>
-    <!-- base of the robot, should be ground level directly below center points of wheels -->
+  <!-- base of the robot, should be ground level directly below center points of wheels -->
   <link name="base_link">
-    <xacro:null_link/>
+  <xacro:null_link/>
   </link>
   <gazebo reference="base_link">
-    <material>Gazebo/Grey</material>
+  <material>Gazebo/Grey</material>
   </gazebo>
   <link name="base_footprint">
-    <xacro:null_link/>
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