Commit message: Added dae files

File: boilerbot_description_integ/urdf/mybot.xacro (robot description, xacro)
@@ -1,25 +1,5 @@
 <?xml version='1.0'?>
 <robot name="myrobot" xmlns:xacro="http://www.ros.org/wiki/xacro">
-  <!--wheels -->
-  <xacro:property name="drive_wheel_diameter" value="0.1651"/>
-  <xacro:property name="drive_wheel_width" value="0.0381"/>
-  <xacro:property name="drive_wheel_mass" value="3.63"/>
-  <xacro:property name="caster_wheel_diameter" value="0.1524"/>
-  <xacro:property name="caster_wheel_width" value="0.0508"/>
-  <xacro:property name="caster_wheel_mass" value="1.81"/>
-  <!--chassis -->
-  <xacro:property name="chassis_length" value="0.50"/>
-  <xacro:property name="chassis_width" value="0.25"/>
-  <xacro:property name="chassis_height" value="0.01"/>
-  <xacro:property name="chassis_mass" value="37"/>
-  <xacro:property name="vehicle_clearance" value="0.25"/>
-  <!--camera -->
-  <xacro:property name="cameraSize" value="0.05"/>
-  <xacro:property name="cameraMass" value="0.03"/>
-  <xacro:property name="camera_mount_height" value="0.5"/>
-  <xacro:property name="camera_mount_width" value="0.05"/>
-  <xacro:property name="camera_mount_length" value="0.05"/>
-  <xacro:property name="camera_mount_mass" value="0.05"/>
-  <!--LiDAR-->
+  <!---->
   <!--INS -->
   <!--Payload -->
@@ -28,208 +8,5 @@
   <xacro:include filename="$(find boilerbot_description_integ)/urdf/materials.xacro" />
   <xacro:include filename="$(find boilerbot_description_integ)/urdf/macros.xacro" />
-  <link name='chassis'>
-    <pose>0 0 0.1 0 0 0</pose>
-    <inertial>
-      <mass value="${chassis_mass}"/>
-      <origin xyz="0.0 0 0.1" rpy=" 0 0 0"/>
-      <inertia
-          ixx="${2 / 5 * chassis_mass * 1 ** 2}" ixy="0" ixz="0"
-          iyy="${2 / 5 * chassis_mass * 1 ** 2}" iyz="0"
-          izz="${2 / 5 * chassis_mass * 1 ** 2}"
-      />
-    </inertial>
-    <collision name='collision'>
-      <geometry>
-        <box size="${chassis_length} ${chassis_width} ${chassis_height}"/>
-      </geometry>
-    </collision>
-    <visual name='chassis_visual'>
-      <origin xyz="0 0 0" rpy=" 0 0 0"/>
-      <geometry>
-        <box size="${chassis_length} ${chassis_width} ${chassis_height}"/>
-      </geometry>
-    </visual>
-  </link>
-  <link name="left_caster">
-    <collision name='left_caster_collision'>
-      <origin xyz="0 0 0" rpy=" 0 0 0"/>
-      <geometry>
-        <cylinder radius="${caster_wheel_diameter/2}" length="${caster_wheel_width}"/>
-      </geometry>
-    </collision>
-    <visual name="left_caster_visual">
-      <origin xyz="0 0 0" rpy="0 1.5707 1.5707"/>
-      <geometry>
-        <cylinder radius="${caster_wheel_diameter/2}" length="${caster_wheel_width}"/>
-      </geometry>
-    </visual>
-    <inertial>
-      <origin xyz="0 0 0" rpy="0 1.5707 1.5707"/>
-      <mass value="${caster_wheel_mass}"/>
-      <cylinder_inertia m="${caster_wheel_mass}" r="${caster_wheel_diameter/2}" h="${drive_wheel_width}"/>
-      <inertia
-        ixx="1.0" ixy="0.0" ixz="0.0"
-        iyy="1.0" iyz="0.0"
-        izz="1.0"/>
-    </inertial>
-  </link>
-  <link name="right_caster">
-    <collision name='right_caster_collision'>
-      <origin xyz="0 0 0" rpy="0 1.5707 1.5707"/>
-      <geometry>
-        <cylinder radius="${caster_wheel_diameter/2}" length="${caster_wheel_width}"/>
-      </geometry>
-    </collision>
-    <visual name="right_caster_visual">
-      <origin xyz="0 0 0" rpy="0 1.5707 1.5707"/>
-      <geometry>
-        <cylinder radius="${caster_wheel_diameter/2}" length="${caster_wheel_width}"/>
-      </geometry>
-    </visual>
-    <inertial>
-      <origin xyz="0 0 0" rpy="0 1.5707 1.5707"/>
-      <mass value="${caster_wheel_mass}"/>
-      <cylinder_inertia m="${caster_wheel_mass}" r="${caster_wheel_diameter/2}" h="${caster_wheel_width}"/>
-      <inertia
-        ixx="1.0" ixy="0.0" ixz="0.0"
-        iyy="1.0" iyz="0.0"
-        izz="1.0"/>
-    </inertial>
-  </link>
-  <link name="left_wheel">
-    <collision name="collision">
-      <origin xyz="0 0 0" rpy="0 1.5707 1.5707"/>
-      <geometry>
-        <cylinder radius="${drive_wheel_diameter/2}" length="${drive_wheel_width}"/>
-      </geometry>
-    </collision>
-    <visual name="left_wheel_visual">
-      <origin xyz="0 0 0" rpy="0 1.5707 1.5707"/>
-      <geometry>
-        <cylinder radius="${drive_wheel_diameter/2}" length="${drive_wheel_width}"/>
-      </geometry>
-    </visual>
-    <inertial>
-      <origin xyz="0 0 0" rpy="0 1.5707 1.5707"/>
-      <mass value="${drive_wheel_mass}"/>
-      <cylinder_inertia m="${drive_wheel_mass}" r="${drive_wheel_diameter/2}" h="${drive_wheel_width}"/>
-      <inertia
-        ixx="1.0" ixy="0.0" ixz="0.0"
-        iyy="1.0" iyz="0.0"
-        izz="1.0"/>
-    </inertial>
-  </link>
-  <link name="right_wheel">
-    <!--origin xyz="0.1 -0.13 0.1" rpy="0 1.5707 1.5707"/-->
-    <collision name="collision">
-      <origin xyz="0 0 0" rpy="0 1.5707 1.5707"/>
-      <geometry>
-        <cylinder radius="${drive_wheel_diameter/2}" length="${drive_wheel_width}"/>
-      </geometry>
-    </collision>
-    <visual name="right_wheel_visual">
-      <origin xyz="0 0 0" rpy="0 1.5707 1.5707"/>
-      <geometry>
-        <cylinder radius="${drive_wheel_diameter/2}" length="${drive_wheel_width}"/>
-      </geometry>
-    </visual>
-    <inertial>
-      <origin xyz="0 0 0" rpy="0 1.5707 1.5707"/>
-      <mass value="5"/>
-      <cylinder_inertia m="${drive_wheel_mass}" r="${drive_wheel_diameter/2}" h="${drive_wheel_width}"/>
-      <inertia
-        ixx="1.0" ixy="0.0" ixz="0.0"
-        iyy="1.0" iyz="0.0"
-        izz="1.0"/>
-    </inertial>
-  </link>
-  <joint type="continuous" name="left_wheel_hinge">
-    <origin xyz="0.2 0.15 0" rpy="0 0 0"/>
-    <child link="left_wheel"/>
-    <parent link="chassis"/>
-    <axis xyz="0 1 0" rpy="0 0 0"/>
-    <limit effort="100" velocity="100"/>
-    <joint_properties damping="0.0" friction="0.0"/>
-  </joint>
-  <joint type="continuous" name="right_wheel_hinge">
-    <origin xyz="0.2 -0.15 0" rpy="0 0 0"/>
-    <child link="right_wheel"/>
-    <parent link="chassis"/>
-    <axis xyz="0 1 0" rpy="0 0 0"/>
-    <limit effort="100" velocity="100"/>
-    <joint_properties damping="0.0" friction="0.0"/>
-  </joint>
-  <joint type="continuous" name="left_caster_hinge">
-    <origin xyz="-0.2 0.15 0" rpy="0 0 0"/>
-    <child link="left_caster"/>
-    <parent link="chassis"/>
-    <axis xyz="0 1 0" rpy="0 0 0"/>
-    <limit effort="100" velocity="100"/>
-    <joint_properties damping="0.0" friction="0.0"/>
-  </joint>
-  <joint type="continuous" name="right_caster_hinge">
-    <origin xyz="-0.2 -0.15 0" rpy="0 0 0"/>
-    <child link="right_caster"/>
-    <parent link="chassis"/>
-    <axis xyz="0 1 0" rpy="0 0 0"/>
-    <limit effort="100" velocity="100"/>
-    <joint_properties damping="0.0" friction="0.0"/>
-  </joint>
-  <link name="camera">
-    <collision>
-      <origin xyz="0 0 0" rpy="0 0 0"/>
-      <geometry>
-        <box size="${cameraSize} ${cameraSize} ${cameraSize}"/>
-      </geometry>
-    </collision>
-    <visual>
-      <origin xyz="0 0 0" rpy="0 0 0"/>
-      <geometry>
-        <box size="${cameraSize} ${cameraSize} ${cameraSize}"/>
-      </geometry>
-      <material name="green"/>
-    </visual>
-    <inertial>
-      <mass value="${cameraMass}" />
-      <origin xyz="0 0 0" rpy="0 0 0"/>
-      <box_inertia m="${cameraMass}" x="${cameraSize}" y="${cameraSize}" z="${cameraSize}" />
-      <inertia ixx="1e-6" ixy="0" ixz="0" iyy="1e-6" iyz="0" izz="1e-6" />
-    </inertial>
-  </link>
-  <link name="camera_mount">
-    <collision>
-      <origin xyz="0 0 0" rpy="0 0 0"/>
-      <geometry>
-        <box size="${camera_mount_length} ${camera_mount_width} ${camera_mount_height}"/>
-      </geometry>
-    </collision>
-    <visual>
-      <origin xyz="0 0 0" rpy="0 0 0"/>
-      <geometry>
-        <box size="${camera_mount_length} ${camera_mount_width} ${camera_mount_height}"/>
-      </geometry>
-      <material name="black"/>
-    </visual>
-    <inertial>
-      <mass value="${camera_mount_mass}" />
-      <origin xyz="0 0 0" rpy="0 0 0"/>
-      <box_inertia m="${camera_mount_mass}" x="${camera_mount_length}" y="${camera_mount_width}" z="${camera_mount_height}" />
-      <inertia ixx="1e-6" ixy="0" ixz="0" iyy="1e-6" iyz="0" izz="1e-6" />
-    </inertial>
-  </link>
-  <joint name="camera_mount_joint" type="fixed">
-    <axis xyz="0 1 0" />
-    <origin xyz="0 0 ${vehicle_clearance}" rpy="0 0 0"/>
-    <parent link="chassis"/>
-    <child link="camera_mount"/>
-  </joint>
-  <joint name="camera_joint" type="fixed">
-    <axis xyz="0 1 0" />
-    <origin xyz="0 0 3" rpy="0 0.8 0"/>
-    <parent link="camera_mount"/>
-    <child link="camera"/>
-  </joint>
-  <!-- Hokuyo Laser -->
-  <link name="hokuyo">
+  <link name="boiler_bot">
     <collision>
       <origin xyz="0 0 0" rpy="0 0 0"/>
@@ -241,5 +18,5 @@
       <origin xyz="0 0 0" rpy="0 0 0"/>
       <geometry>
-        <mesh filename="package://boilerbot_description_integ/meshes/hokuyo.dae"/>
+        <mesh filename="package://boilerbot_description_integ/meshes/bb10_model.dae"/>
       </geometry>
     </visual>
@@ -250,9 +27,3 @@
     </inertial>
   </link>
-  <joint name="hokuyo_joint" type="fixed">
-    <axis xyz="0 1 0" />
-    <origin xyz=".15 0 .1" rpy="0 0 0"/>
-    <parent link="chassis"/>
-    <child link="hokuyo"/>
-  </joint>
 </robot>

Commit message: Fixed the dae file to have the correct units and transforms

File: boilerbot_description_integ/urdf/mybot.xacro (robot description, xacro)
@@ -18,5 +18,5 @@
       <origin xyz="0 0 0" rpy="0 0 0"/>
       <geometry>
-        <mesh filename="package://boilerbot_description_integ/meshes/bb10_model.dae"/>
+        <mesh filename="package://boilerbot_description_integ/meshes/bb10_no_wheels.dae"/>
       </geometry>
     </visual>

Commit message: Added xacro file

File: boilerbot_description_integ/urdf/mybot.xacro (robot description, xacro)
@@ -1,5 +1,25 @@
 <?xml version='1.0'?>
 <robot name="myrobot" xmlns:xacro="http://www.ros.org/wiki/xacro">
-  <!---->
+  <!--wheels -->
+  <xacro:property name="drive_wheel_diameter" value="0.1651"/>
+  <xacro:property name="drive_wheel_width" value="0.0381"/>
+  <xacro:property name="drive_wheel_mass" value="3.63"/>
+  <xacro:property name="caster_wheel_diameter" value="0.1524"/>
+  <xacro:property name="caster_wheel_width" value="0.0508"/>
+  <xacro:property name="caster_wheel_mass" value="1.81"/>
+  <!--chassis -->
+  <xacro:property name="chassis_length" value="0.50"/>
+  <xacro:property name="chassis_width" value="0.25"/>
+  <xacro:property name="chassis_height" value="0.01"/>
+  <xacro:property name="chassis_mass" value="37"/>
+  <xacro:property name="vehicle_clearance" value="0.25"/>
+  <!--camera -->
+  <xacro:property name="cameraSize" value="0.05"/>
+  <xacro:property name="cameraMass" value="0.03"/>
+  <xacro:property name="camera_mount_height" value="0.5"/>
+  <xacro:property name="camera_mount_width" value="0.05"/>
+  <xacro:property name="camera_mount_length" value="0.05"/>
+  <xacro:property name="camera_mount_mass" value="0.05"/>
+  <!--LiDAR-->
   <!--INS -->
   <!--Payload -->
@@ -8,8 +28,211 @@
   <xacro:include filename="$(find boilerbot_description_integ)/urdf/materials.xacro" />
   <xacro:include filename="$(find boilerbot_description_integ)/urdf/macros.xacro" />
-  <link name="boiler_bot">
+  <link name='chassis'>
+    <pose>0 0 0.1 0 0 0</pose>
+    <inertial>
+      <mass value="${chassis_mass}"/>
+      <origin xyz="0.0 0 0.1" rpy=" 0 0 0"/>
+      <inertia
+          ixx="${2 / 5 * chassis_mass * 1 ** 2}" ixy="0" ixz="0"
+          iyy="${2 / 5 * chassis_mass * 1 ** 2}" iyz="0"
+          izz="${2 / 5 * chassis_mass * 1 ** 2}"
+      />
+    </inertial>
+    <collision name='collision'>
+      <geometry>
+        <box size="${chassis_length} ${chassis_width} ${chassis_height}"/>
+      </geometry>
+    </collision>
+    <visual name='chassis_visual'>
+      <origin xyz="0 0 0" rpy=" 0 0 0"/>
+      <geometry>
+        <box size="${chassis_length} ${chassis_width} ${chassis_height}"/>
+      </geometry>
+    </visual>
+  </link>
+  <link name="left_castor_wheel">
+    <collision name='left_caster_collision'>
+      <origin xyz="0 0 0" rpy=" 0 0 0"/>
+      <geometry>
+        <cylinder radius="${caster_wheel_diameter/2}" length="${caster_wheel_width}"/>
+      </geometry>
+    </collision>
+    <visual name="left_caster_visual">
+      <origin xyz="0 0 0" rpy="0 1.5707 1.5707"/>
+      <geometry>
+        <cylinder radius="${caster_wheel_diameter/2}" length="${caster_wheel_width}"/>
+      </geometry>
+    </visual>
+    <inertial>
+      <origin xyz="0 0 0" rpy="0 1.5707 1.5707"/>
+      <mass value="${caster_wheel_mass}"/>
+      <cylinder_inertia m="${caster_wheel_mass}" r="${caster_wheel_diameter/2}" h="${drive_wheel_width}"/>
+      <inertia
+        ixx="1.0" ixy="0.0" ixz="0.0"
+        iyy="1.0" iyz="0.0"
+        izz="1.0"/>
+    </inertial>
+  </link>
+  <link name="right_castor_wheel">
+    <collision name='right_caster_collision'>
+      <origin xyz="0 0 0" rpy="0 1.5707 1.5707"/>
+      <geometry>
+        <cylinder radius="${caster_wheel_diameter/2}" length="${caster_wheel_width}"/>
+      </geometry>
+    </collision>
+    <visual name="right_caster_visual">
+      <origin xyz="0 0 0" rpy="0 1.5707 1.5707"/>
+      <geometry>
+        <cylinder radius="${caster_wheel_diameter/2}" length="${caster_wheel_width}"/>
+      </geometry>
+    </visual>
+    <inertial>
+      <origin xyz="0 0 0" rpy="0 1.5707 1.5707"/>
+      <mass value="${caster_wheel_mass}"/>
+      <cylinder_inertia m="${caster_wheel_mass}" r="${caster_wheel_diameter/2}" h="${caster_wheel_width}"/>
+      <inertia
+        ixx="1.0" ixy="0.0" ixz="0.0"
+        iyy="1.0" iyz="0.0"
+        izz="1.0"/>
+    </inertial>
+  </link>
+  <link name="left_drive_wheel">
+    <collision name="collision">
+      <origin xyz="0 0 0" rpy="0 1.5707 1.5707"/>
+      <geometry>
+        <cylinder radius="${drive_wheel_diameter/2}" length="${drive_wheel_width}"/>
+      </geometry>
+    </collision>
+    <visual name="left_wheel_visual">
+      <origin xyz="0 0 0" rpy="0 1.5707 1.5707"/>
+      <geometry>
+        <cylinder radius="${drive_wheel_diameter/2}" length="${drive_wheel_width}"/>
+      </geometry>
+    </visual>
+    <inertial>
+      <origin xyz="0 0 0" rpy="0 1.5707 1.5707"/>
+      <mass value="${drive_wheel_mass}"/>
+      <cylinder_inertia m="${drive_wheel_mass}" r="${drive_wheel_diameter/2}" h="${drive_wheel_width}"/>
+      <inertia
+        ixx="1.0" ixy="0.0" ixz="0.0"
+        iyy="1.0" iyz="0.0"
+        izz="1.0"/>
+    </inertial>
+  </link>
+  <link name="right_drive_wheel">
+    <!--origin xyz="0.1 -0.13 0.1" rpy="0 1.5707 1.5707"/-->
+    <collision name="collision">
+      <origin xyz="0 0 0" rpy="0 1.5707 1.5707"/>
+      <geometry>
+        <cylinder radius="${drive_wheel_diameter/2}" length="${drive_wheel_width}"/>
+      </geometry>
+    </collision>
+    <visual name="right_wheel_visual">
+      <origin xyz="0 0 0" rpy="0 1.5707 1.5707"/>
+      <geometry>
+        <cylinder radius="${drive_wheel_diameter/2}" length="${drive_wheel_width}"/>
+      </geometry>
+    </visual>
+    <inertial>
+      <origin xyz="0 0 0" rpy="0 1.5707 1.5707"/>
+      <mass value="5"/>
+      <cylinder_inertia m="${drive_wheel_mass}" r="${drive_wheel_diameter/2}" h="${drive_wheel_width}"/>
+      <inertia
+        ixx="1.0" ixy="0.0" ixz="0.0"
+        iyy="1.0" iyz="0.0"
+        izz="1.0"/>
+    </inertial>
+  </link>
+  <joint type="continuous" name="left_drive_hinge">
+    <origin xyz="0.2 0.15 0" rpy="0 0 0"/>
+    <child link="left_wheel"/>
+    <parent link="chassis"/>
+    <axis xyz="0 1 0" rpy="0 0 0"/>
+    <limit effort="100" velocity="100"/>
+    <joint_properties damping="0.0" friction="0.0"/>
+  </joint>
+  <joint type="continuous" name="right_drive_hinge">
+    <origin xyz="0.2 -0.15 0" rpy="0 0 0"/>
+    <child link="right_wheel"/>
+    <parent link="chassis"/>
+    <axis xyz="0 1 0" rpy="0 0 0"/>
+    <limit effort="100" velocity="100"/>
+    <joint_properties damping="0.0" friction="0.0"/>
+  </joint>
+  <joint type="continuous" name="left_castor_hinge">
+    <origin xyz="-0.2 0.15 0" rpy="0 0 0"/>
+    <child link="left_caster"/>
+    <parent link="chassis"/>
+    <axis xyz="0 1 0" rpy="0 0 0"/>
+    <limit effort="100" velocity="100"/>
+    <joint_properties damping="0.0" friction="0.0"/>
+  </joint>
+  <joint type="continuous" name="right_castor_hinge">
+    <origin xyz="-0.2 -0.15 0" rpy="0 0 0"/>
+    <child link="right_caster"/>
+    <parent link="chassis"/>
+    <axis xyz="0 1 0" rpy="0 0 0"/>
+    <limit effort="100" velocity="100"/>
+    <joint_properties damping="0.0" friction="0.0"/>
+  </joint>
+  <link name="camera">
     <collision>
       <origin xyz="0 0 0" rpy="0 0 0"/>
       <geometry>
+        <box size="${cameraSize} ${cameraSize} ${cameraSize}"/>
+      </geometry>
+    </collision>
+    <visual>
+      <origin xyz="0 0 0" rpy="0 0 0"/>
+      <geometry>
+        <box size="${cameraSize} ${cameraSize} ${cameraSize}"/>
+      </geometry>
+      <material name="green"/>
+    </visual>
+    <inertial>
+      <mass value="${cameraMass}" />
+      <origin xyz="0 0 0" rpy="0 0 0"/>
+      <box_inertia m="${cameraMass}" x="${cameraSize}" y="${cameraSize}" z="${cameraSize}" />
+      <inertia ixx="1e-6" ixy="0" ixz="0" iyy="1e-6" iyz="0" izz="1e-6" />
+    </inertial>
+  </link>
+  <link name="camera_mount">
+    <collision>
+      <origin xyz="0 0 0" rpy="0 0 0"/>
+      <geometry>
+        <box size="${camera_mount_length} ${camera_mount_width} ${camera_mount_height}"/>
+      </geometry>
+    </collision>
+    <visual>
+      <origin xyz="0 0 0" rpy="0 0 0"/>
+      <geometry>
+        <box size="${camera_mount_length} ${camera_mount_width} ${camera_mount_height}"/>
+      </geometry>
+      <material name="black"/>
+    </visual>
+    <inertial>
+      <mass value="${camera_mount_mass}" />
+      <origin xyz="0 0 0" rpy="0 0 0"/>
+      <box_inertia m="${camera_mount_mass}" x="${camera_mount_length}" y="${camera_mount_width}" z="${camera_mount_height}" />
+      <inertia ixx="1e-6" ixy="0" ixz="0" iyy="1e-6" iyz="0" izz="1e-6" />
+    </inertial>
+  </link>
+  <joint name="camera_mount_joint" type="fixed">
+    <axis xyz="0 1 0" />
+    <origin xyz="0 0 ${vehicle_clearance}" rpy="0 0 0"/>
+    <parent link="chassis"/>
+    <child link="camera_mount"/>
+  </joint>
+  <joint name="camera_joint" type="fixed">
+    <axis xyz="0 1 0" />
+    <origin xyz="0 0 3" rpy="0 0.8 0"/>
+    <parent link="camera_mount"/>
+    <child link="camera"/>
+  </joint>
+  <!-- Hokuyo Laser -->
+  <link name="hokuyo">
+    <collision>
+      <origin xyz="0 0 0" rpy="0 0 0"/>
+      <geometry>
     <box size="0.1 0.1 0.1"/>
       </geometry>
@@ -18,5 +241,5 @@
       <origin xyz="0 0 0" rpy="0 0 0"/>
       <geometry>
-        <mesh filename="package://boilerbot_description_integ/meshes/bb10_no_wheels.dae"/>
+        <mesh filename="package://boilerbot_description_integ/meshes/hokuyo.dae"/>
       </geometry>
     </visual>
@@ -27,3 +250,9 @@
     </inertial>
   </link>
+  <joint name="hokuyo_joint" type="fixed">
+    <axis xyz="0 1 0" />
+    <origin xyz=".15 0 .1" rpy="0 0 0"/>
+    <parent link="chassis"/>
+    <child link="hokuyo"/>
+  </joint>
 </robot>
