Commit message: Robot moving, near working slam implementation

File: boilerbot_description_integ/urdf/mybot.xacro (robot description, xacro)
@@ -15,5 +15,5 @@
   <xacro:property name="vehicle_clearance" value="0.25"/>
   <!--camera -->
-  <xacro:property name="cameraSize" value="0.05"/>
+  <xacro:property name="cameraSize" value="0.01"/>
   <xacro:property name="cameraMass" value="0.03"/>
   <xacro:property name="camera_mount_height" value="0.5"/>
@@ -21,13 +21,10 @@
   <xacro:property name="camera_mount_length" value="0.05"/>
   <xacro:property name="camera_mount_mass" value="0.05"/>
-  <!--LiDAR-->
-  <!--INS -->
-  <!--Payload -->
-   <!--Laptop -->
   <xacro:include filename="$(find boilerbot_description_integ)/urdf/mybot.gazebo" />
   <xacro:include filename="$(find boilerbot_description_integ)/urdf/materials.xacro" />
   <xacro:include filename="$(find boilerbot_description_integ)/urdf/macros.xacro" />
+  <!-- Chassis Link -->
   <link name='chassis'>
-    <pose>0 0 0.1 0 0 0</pose>
+    <pose>0 0 0 0 0 0</pose>
     <inertial>
       <mass value="${chassis_mass}"/>
@@ -41,14 +38,15 @@
     <collision name='collision'>
       <geometry>
-        <box size="${chassis_length} ${chassis_width} ${chassis_height}"/>
+        <mesh filename="package://boilerbot_description_integ/meshes/bodyNoWheels.dae"/>
       </geometry>
     </collision>
     <visual name='chassis_visual'>
-      <origin xyz="0 0 0" rpy=" 0 0 0"/>
-      <geometry>
-        <box size="${chassis_length} ${chassis_width} ${chassis_height}"/>
-      </geometry>
-    </visual>
-  </link>
+      <origin xyz="0 0 0" rpy=" 0 0 -1.5707"/>
+      <geometry>
+        <mesh filename="package://boilerbot_description_integ/meshes/bodyNoWheels.dae"/>
+      </geometry>
+    </visual>
+  </link>
+  <!-- Left Castor Wheel Link -->
   <link name="left_castor_wheel">
     <collision name='left_caster_collision'>
@@ -74,4 +72,5 @@
     </inertial>
   </link>
+  <!-- Right Castor Wheel Link -->
   <link name="right_castor_wheel">
     <collision name='right_caster_collision'>
@@ -97,4 +96,5 @@
     </inertial>
   </link>
+  <!-- Left Drive Wheel Link -->
   <link name="left_drive_wheel">
     <collision name="collision">
@@ -120,4 +120,5 @@
     </inertial>
   </link>
+  <!-- Right Drive Wheel Link -->
   <link name="right_drive_wheel">
     <!--origin xyz="0.1 -0.13 0.1" rpy="0 1.5707 1.5707"/-->
@@ -136,5 +137,5 @@
     <inertial>
       <origin xyz="0 0 0" rpy="0 1.5707 1.5707"/>
-      <mass value="5"/>
+      <mass value="${drive_wheel_mass}"/>
       <cylinder_inertia m="${drive_wheel_mass}" r="${drive_wheel_diameter/2}" h="${drive_wheel_width}"/>
       <inertia
@@ -144,36 +145,41 @@
     </inertial>
   </link>
+  <!-- Left Drive wheel joint -->
   <joint type="continuous" name="left_drive_hinge">
-    <origin xyz="0.2 0.15 0" rpy="0 0 0"/>
-    <child link="left_wheel"/>
-    <parent link="chassis"/>
-    <axis xyz="0 1 0" rpy="0 0 0"/>
-    <limit effort="100" velocity="100"/>
-    <joint_properties damping="0.0" friction="0.0"/>
-  </joint>
+    <origin xyz="0 0.31 0.1" rpy="0 0 0"/>
+    <child link="left_drive_wheel"/>
+    <parent link="chassis"/>
+    <axis xyz="0 1 0" rpy="0 0 0"/>
+    <limit effort="100" velocity="100"/>
+    <joint_properties damping="0.0" friction="0.0"/>
+  </joint>
+  <!-- Right Drive Wheel Joint -->
   <joint type="continuous" name="right_drive_hinge">
-    <origin xyz="0.2 -0.15 0" rpy="0 0 0"/>
-    <child link="right_wheel"/>
-    <parent link="chassis"/>
-    <axis xyz="0 1 0" rpy="0 0 0"/>
-    <limit effort="100" velocity="100"/>
-    <joint_properties damping="0.0" friction="0.0"/>
-  </joint>
+    <origin xyz="0 -0.31 0.1" rpy="0 0 0"/>
+    <child link="right_drive_wheel"/>
+    <parent link="chassis"/>
+    <axis xyz="0 1 0" rpy="0 0 0"/>
+    <limit effort="100" velocity="100"/>
+    <joint_properties damping="0.0" friction="0.0"/>
+  </joint>
+  <!-- Left Castor Wheel Joint -->
   <joint type="continuous" name="left_castor_hinge">
-    <origin xyz="-0.2 0.15 0" rpy="0 0 0"/>
-    <child link="left_caster"/>
-    <parent link="chassis"/>
-    <axis xyz="0 1 0" rpy="0 0 0"/>
-    <limit effort="100" velocity="100"/>
-    <joint_properties damping="0.0" friction="0.0"/>
-  </joint>
+    <origin xyz="-0.53 0.13 0.09" rpy="0 0 0"/>
+    <child link="left_castor_wheel"/>
+    <parent link="chassis"/>
+    <axis xyz="0 1 0" rpy="0 0 0"/>
+    <limit effort="100" velocity="100"/>
+    <joint_properties damping="0.0" friction="0.0"/>
+  </joint>
+  <!-- Right Castor Wheel Joint -->
   <joint type="continuous" name="right_castor_hinge">
-    <origin xyz="-0.2 -0.15 0" rpy="0 0 0"/>
-    <child link="right_caster"/>
-    <parent link="chassis"/>
-    <axis xyz="0 1 0" rpy="0 0 0"/>
-    <limit effort="100" velocity="100"/>
-    <joint_properties damping="0.0" friction="0.0"/>
-  </joint>
+    <origin xyz="-0.53 -0.13 0.09" rpy="0 0 0"/>
+    <child link="right_castor_wheel"/>
+    <parent link="chassis"/>
+    <axis xyz="0 1 0" rpy="0 0 0"/>
+    <limit effort="100" velocity="100"/>
+    <joint_properties damping="0.0" friction="0.0"/>
+  </joint>
+  <!-- Camera -->
   <link name="camera">
     <collision>
@@ -197,35 +203,8 @@
     </inertial>
   </link>
-  <link name="camera_mount">
-    <collision>
-      <origin xyz="0 0 0" rpy="0 0 0"/>
-      <geometry>
-        <box size="${camera_mount_length} ${camera_mount_width} ${camera_mount_height}"/>
-      </geometry>
-    </collision>
-    <visual>
-      <origin xyz="0 0 0" rpy="0 0 0"/>
-      <geometry>
-        <box size="${camera_mount_length} ${camera_mount_width} ${camera_mount_height}"/>
-      </geometry>
-      <material name="black"/>
-    </visual>
-    <inertial>
-      <mass value="${camera_mount_mass}" />
-      <origin xyz="0 0 0" rpy="0 0 0"/>
-      <box_inertia m="${camera_mount_mass}" x="${camera_mount_length}" y="${camera_mount_width}" z="${camera_mount_height}" />
-      <inertia ixx="1e-6" ixy="0" ixz="0" iyy="1e-6" iyz="0" izz="1e-6" />
-    </inertial>
-  </link>
-  <joint name="camera_mount_joint" type="fixed">
-    <axis xyz="0 1 0" />
-    <origin xyz="0 0 ${vehicle_clearance}" rpy="0 0 0"/>
-    <parent link="chassis"/>
-    <child link="camera_mount"/>
-  </joint>
   <joint name="camera_joint" type="fixed">
     <axis xyz="0 1 0" />
-    <origin xyz="0 0 3" rpy="0 0.8 0"/>
-    <parent link="camera_mount"/>
+    <origin xyz="-0.04 0 1.05" rpy="0 0.5 0"/>
+    <parent link="chassis"/>
     <child link="camera"/>
   </joint>
@@ -252,5 +231,5 @@
   <joint name="hokuyo_joint" type="fixed">
     <axis xyz="0 1 0" />
-    <origin xyz=".15 0 .1" rpy="0 0 0"/>
+    <origin xyz="0.25 0 .457" rpy="0 0 0"/>
     <parent link="chassis"/>
     <child link="hokuyo"/>

File: boilerbot_description_integ/urdf/mybot_new.xacro (robot description, xacro)
@@ -12,8 +12,9 @@
   <xacro:include filename="$(find boilerbot_description_integ)/urdf/macros.xacro" />
   <link name="chassis">
+    <pose>0 0 0 0 0</pose>
     <collision>
       <origin xyz="0 0 0" rpy="0 0 0"/>
       <geometry>
-    <box size="0.1 0.1 0.1"/>
+    	<box size="0.1 0.1 0.1"/>
       </geometry>
     </collision>
@@ -27,5 +28,5 @@
       <mass value="76.65" />
       <origin xyz="0 0 0" rpy="0 0 0"/>
-      <inertia ixx="50" ixy="0" ixz="0" iyy="50" iyz="0" izz="50" />
+      <inertia ixx="1" ixy="0" ixz="0" iyy="1" iyz="0" izz="1" />
     </inertial>
   </link>
@@ -35,5 +36,5 @@
       <origin xyz="0 0 0" rpy="0 0 0"/>
       <geometry>
-    <box size="0.1 0.1 0.1"/>
+        <mesh filename="package://boilerbot_description_integ/meshes/driveWheelLeft.dae"/>
       </geometry>
     </collision>
@@ -63,5 +64,5 @@
       <origin xyz="0 0 0" rpy="0 0 0"/>
       <geometry>
-    <box size="0.1 0.1 0.1"/>
+        <mesh filename="package://boilerbot_description_integ/meshes/driveWheelRight.dae"/>
       </geometry>
     </collision>
@@ -91,5 +92,5 @@
       <origin xyz="0 0 0" rpy="0 0 0"/>
       <geometry>
-    <box size="0.1 0.1 0.1"/>
+        <mesh filename="package://boilerbot_description_integ/meshes/castorLeft.dae"/>
       </geometry>
     </collision>
@@ -119,5 +120,5 @@
       <origin xyz="0 0 0" rpy="0 0 0"/>
       <geometry>
-    <box size="0.1 0.1 0.1"/>
+        <mesh filename="package://boilerbot_description_integ/meshes/castorRight.dae"/>
       </geometry>
     </collision>
@@ -145,5 +146,5 @@
   <link name="camera">
     <collision>
-      <origin xyz="0 0 -0.1" rpy="0 0 0"/>
+      <origin xyz="0 0 0" rpy="0 0 0"/>
       <geometry>
         <box size="0.1 0.01 0.1"/>
@@ -175,5 +176,5 @@
       <origin xyz="0 0 0" rpy="0 0 0"/>
       <geometry>
-    <box size="0.1 0.1 0.1"/>
+    	<box size="0.1 0.1 0.1"/>
       </geometry>
     </collision>

Commit message: Tweaked the lidar height and angle to appropriate values

File: boilerbot_description_integ/urdf/mybot.xacro (robot description, xacro)
@@ -2,15 +2,15 @@
 <robot name="myrobot" xmlns:xacro="http://www.ros.org/wiki/xacro">
   <!--wheels -->
-  <xacro:property name="drive_wheel_diameter" value="0.1651"/>
+  <xacro:property name="drive_wheel_diameter" value="0.1811"/>
   <xacro:property name="drive_wheel_width" value="0.0381"/>
-  <xacro:property name="drive_wheel_mass" value="3.63"/>
-  <xacro:property name="caster_wheel_diameter" value="0.1524"/>
+  <xacro:property name="drive_wheel_mass" value="2.5"/>
+  <xacro:property name="caster_wheel_diameter" value="0.1811"/>
   <xacro:property name="caster_wheel_width" value="0.0508"/>
-  <xacro:property name="caster_wheel_mass" value="1.81"/>
+  <xacro:property name="caster_wheel_mass" value="2.5"/>
   <!--chassis -->
   <xacro:property name="chassis_length" value="0.50"/>
   <xacro:property name="chassis_width" value="0.25"/>
   <xacro:property name="chassis_height" value="0.01"/>
-  <xacro:property name="chassis_mass" value="37"/>
+  <xacro:property name="chassis_mass" value="25"/>
   <xacro:property name="vehicle_clearance" value="0.25"/>
   <!--camera -->
@@ -25,9 +25,12 @@
   <xacro:include filename="$(find boilerbot_description_integ)/urdf/macros.xacro" />
   <!-- Chassis Link -->
+  <link name='base_link'>
+    <pose>0 0 0 0 0 0</pose>
+  </link>
   <link name='chassis'>
     <pose>0 0 0 0 0 0</pose>
     <inertial>
       <mass value="${chassis_mass}"/>
-      <origin xyz="0.0 0 0.1" rpy=" 0 0 0"/>
+      <origin xyz="0.0 0 0" rpy=" 0 0 0"/>
       <inertia
           ixx="${2 / 5 * chassis_mass * 1 ** 2}" ixy="0" ixz="0"
@@ -48,4 +51,6 @@
     </visual>
   </link>
+  <!-- Payload -->
+  <!--<link name="payload">-->
   <!-- Left Castor Wheel Link -->
   <link name="left_castor_wheel">
@@ -145,9 +150,16 @@
     </inertial>
   </link>
+  <!-- Base Link Chassis joint -->
+  <joint type="fixed" name="base_link_chassis">
+    <origin xyz="0 0 -0.1" rpy="0 0 0"/>
+    <child link="chassis"/>
+    <parent link="base_link"/>
+    <axis xyz="0 1 0"/>
+  </joint>
   <!-- Left Drive wheel joint -->
   <joint type="continuous" name="left_drive_hinge">
-    <origin xyz="0 0.31 0.1" rpy="0 0 0"/>
+    <origin xyz="0 0.31 0" rpy="0 0 0"/>
     <child link="left_drive_wheel"/>
-    <parent link="chassis"/>
+    <parent link="base_link"/>
     <axis xyz="0 1 0" rpy="0 0 0"/>
     <limit effort="100" velocity="100"/>
@@ -156,7 +168,7 @@
   <!-- Right Drive Wheel Joint -->
   <joint type="continuous" name="right_drive_hinge">
-    <origin xyz="0 -0.31 0.1" rpy="0 0 0"/>
+    <origin xyz="0 -0.31 0" rpy="0 0 0"/>
     <child link="right_drive_wheel"/>
-    <parent link="chassis"/>
+    <parent link="base_link"/>
     <axis xyz="0 1 0" rpy="0 0 0"/>
     <limit effort="100" velocity="100"/>
@@ -165,7 +177,7 @@
   <!-- Left Castor Wheel Joint -->
   <joint type="continuous" name="left_castor_hinge">
-    <origin xyz="-0.53 0.13 0.09" rpy="0 0 0"/>
+    <origin xyz="-0.53 0.13 0" rpy="0 0 0"/>
     <child link="left_castor_wheel"/>
-    <parent link="chassis"/>
+    <parent link="base_link"/>
     <axis xyz="0 1 0" rpy="0 0 0"/>
     <limit effort="100" velocity="100"/>
@@ -174,7 +186,7 @@
   <!-- Right Castor Wheel Joint -->
   <joint type="continuous" name="right_castor_hinge">
-    <origin xyz="-0.53 -0.13 0.09" rpy="0 0 0"/>
+    <origin xyz="-0.53 -0.13 0" rpy="0 0 0"/>
     <child link="right_castor_wheel"/>
-    <parent link="chassis"/>
+    <parent link="base_link"/>
     <axis xyz="0 1 0" rpy="0 0 0"/>
     <limit effort="100" velocity="100"/>
@@ -205,6 +217,6 @@
   <joint name="camera_joint" type="fixed">
     <axis xyz="0 1 0" />
-    <origin xyz="-0.04 0 1.05" rpy="0 0.5 0"/>
-    <parent link="chassis"/>
+    <origin xyz="-0.04 0 0.95" rpy="0 0.5 0"/>
+    <parent link="base_link"/>
     <child link="camera"/>
   </joint>
@@ -231,6 +243,6 @@
   <joint name="hokuyo_joint" type="fixed">
     <axis xyz="0 1 0" />
-    <origin xyz="0.25 0 .457" rpy="0 0 0"/>
-    <parent link="chassis"/>
+    <origin xyz="0.25 0 .420" rpy="0 0 0"/>
+    <parent link="base_link"/>
     <child link="hokuyo"/>
   </joint>

Commit message: Made the castor wheels heavier to prevent robot from jerking when coming to a stop

File: boilerbot_description_integ/urdf/mybot.xacro (robot description, xacro)
@@ -7,5 +7,5 @@
   <xacro:property name="caster_wheel_diameter" value="0.1811"/>
   <xacro:property name="caster_wheel_width" value="0.0508"/>
-  <xacro:property name="caster_wheel_mass" value="2.5"/>
+  <xacro:property name="caster_wheel_mass" value="3.7"/>
   <!--chassis -->
   <xacro:property name="chassis_length" value="0.50"/>
